File: riskybirdv3_connector/riskybirdv3_connector.kicad_sch (KiCad schematic)
At the start: 42 parts, among them U15 FT2232HL-REEL, U9 FT2232HL-REEL, Y2 f, Y3 f

Commit message: add: usbs and charger to connector board
Parts:
- added C1, C2: 10n, symbol Device:C_Small
- added C10, C11: 4.7u, Capacitor_SMD:C_0201_0603Metric, symbol Device:C
- added C3, C4, C5, C6: 10u, symbol Device:C_Small
- added D7: LED_RED, LED_SMD:LED_0402_1005Metric, symbol Device:LED
- added F1, F2, F3: 6V 2A, symbol Device:Fuse
- added J1, J2: USB_C_Receptacle_USB2.0_16P, symbol Connector:USB_C_Receptacle_USB2.0_16P
- added J17: Conn_02x12_Odd_Even_MountingPin, riskybird:5037762410, symbol Connector_Generic_MountingPin:Conn_02x12_Odd_Even_MountingPin
- added J4: USB_C_Receptacle_PowerOnly_6P, symbol Connector:USB_C_Receptacle_PowerOnly_6P
- added J7: Conn_01x02, Connector_PinHeader_2.00mm:PinHeader_1x02_P2.00mm_Vertical, symbol Connector_Generic:Conn_01x02
- added R1, R15, R16, R2, R3, R4: 5k1, symbol Device:R_Small
- added R13: 2k, Resistor_SMD:R_0201_0603Metric, symbol Device:R
- added R14: 1k, Resistor_SMD:R_0201_0603Metric, symbol Device:R
- added R5, R6, R8, R9: 22R, symbol Device:R_Small
- added U1, U2: AP2112K-3.3, Package_TO_SOT_SMD:SOT-23-5, symbol Regulator_Linear:AP2112K-3.3
- added U4: MCP73831-2-OT, Package_TO_SOT_SMD:SOT-23-5, symbol riskybird-rescue:MCP73831-2-OT-Battery_Management
Connections:
- net FTDI_3v3_1: now also C4.1, U1.5 (VOUT)
- net FTDI_3v3_2: now also C6.1, U2.5 (VOUT)
- net GND: now also C1.2, C10.2, C2.2, C3.2, C4.2, C5.2, C6.2, J1.A1 (GND), J1.A12 (GND), J1.B1 (GND), J1.B12 (GND), J1.SH (SHIELD), J17.MP (MountPin), J2.A1 (GND), J2.A12 (GND), J2.B1 (GND), J2.B12 (GND), J2.SH (SHIELD), J4.A12 (GND), J4.B12 (GND), J4.SH (SHIELD), J7.2 (Pin_2), R1.2, R13.2, R15.2, R16.2, R2.2, R3.2, R4.2, U1.2 (GND), U2.2 (GND), U4.2 (VSS)
- net NSRST_1: now also J17.10 (Pin_10)
- net NSRST_2: now also J17.9 (Pin_9)
- net NTRST_1: now also J17.12 (Pin_12)
- net NTRST_2: now also J17.11 (Pin_11)
- net RXD_1: now also J17.14 (Pin_14)
- net RXD_2: now also J17.13 (Pin_13)
- net TCK_1: now also J17.2 (Pin_2)
- net TCK_2: now also J17.1 (Pin_1)
- net TDI_1: now also J17.4 (Pin_4)
- net TDI_2: now also J17.3 (Pin_3)
- net TDO_1: now also J17.6 (Pin_6)
- net TDO_2: now also J17.5 (Pin_5)
- net TMS_1: now also J17.8 (Pin_8)
- net TMS_2: now also J17.7 (Pin_7)
- net TXD_1: now also J17.16 (Pin_16)
- net TXD_2: now also J17.15 (Pin_15)
- net USB_DM_2: now also R6.2
- net USB_DP_1: now also R8.2
- net USB_DP_2: now also R9.2
- net USP_DM_1 renamed USB_DM_1
- net USB_DM_1: now also R5.2
- new net: J1.A5 (CC1), R1.1
- new net: J4.A5 (CC1), R15.1
- new net: F3.1, J4.A9 (VBUS), J4.B9 (VBUS)
- new net: J4.B5 (CC2), R16.1
- new net: J1.B5 (CC2), R3.1
- new net: C2.1, F2.1, J2.A4 (VBUS), J2.A9 (VBUS), J2.B4 (VBUS), J2.B9 (VBUS)
- new net: J2.A7 (D-), J2.B7 (D-), R6.1
- new net: J1.A7 (D-), J1.B7 (D-), R5.1
- new net: J2.B5 (CC2), R4.1
- new net: R13.1, U4.5 (PROG)
- new net: D7.1 (K), U4.1 (STAT)
- new net: D7.2 (A), R14.2
- new net: C1.1, F1.1, J1.A4 (VBUS), J1.A9 (VBUS), J1.B4 (VBUS), J1.B9 (VBUS)
- new net: J1.A6 (D+), J1.B6 (D+), R8.1
- new net: J2.A5 (CC1), R2.1
- new net: J2.A6 (D+), J2.B6 (D+), R9.1
- new net: C11.2, U4.3 (VBAT)
- new net +BATT: C11.1, J7.1 (Pin_1)
- new net 5V_1: C3.1, F1.2, U1.1 (VIN), U1.3 (EN)
- new net 5V_2: C5.1, F2.2, U2.1 (VIN), U2.3 (EN)
- new net 5V_3: C10.1, F3.2, R14.1, U4.4 (VDD)
- no-connect marks 46 -> 58
Other:
- note added: "Charger"
- moved on the sheet: C38, C39, C49, C50, C76, C78, R65, R67, U15
