File: riskybirdv3_connector/riskybirdv3_connector.kicad_pcb (KiCad board)
At the start: 4 copper layers, 34.7 x 37 mm, 75 parts, among them J1 USB_C_Receptacle_USB2.0_16P, J2 USB_C_Receptacle_USB2.0_16P, J3 Conn_02x10_Odd_Even, U1 AP2112K-3.3, U15 FT2232HL-REEL, U2 AP2112K-3.3, U9 FT2232HL-REEL, Y2 f, Y3 f

Commit message: add: layout done
Parts:
- added TP12: TestPoint, TestPoint:TestPoint_Pad_D1.0mm, F.Cu at (60.9, 74.5)
- added TP13: TestPoint, TestPoint:TestPoint_Pad_D1.0mm, F.Cu at (37.6, 78.3)
- added TP14: TestPoint, TestPoint:TestPoint_Pad_D1.0mm, F.Cu at (42.3, 100.3)
- added TP16: TestPoint, TestPoint:TestPoint_Pad_D1.0mm, F.Cu at (60.9, 72.0)
- added TP17: TestPoint, TestPoint:TestPoint_Pad_D1.0mm, F.Cu at (32.7, 87.2)
- added TP18: TestPoint, TestPoint:TestPoint_Pad_D1.0mm, F.Cu at (60.9, 69.4)
- added TP19: TestPoint, TestPoint:TestPoint_Pad_D1.0mm, F.Cu at (60.8, 67.0)
- added TP20: TestPoint, TestPoint:TestPoint_Pad_D1.0mm, F.Cu at (60.9, 76.6)
- added TP22: TestPoint, TestPoint:TestPoint_Pad_D1.0mm, F.Cu at (39.6, 77.1)
- added TP23: TestPoint, TestPoint:TestPoint_Pad_D1.0mm, F.Cu at (32.7, 83.8)
- added TP24: TestPoint, TestPoint:TestPoint_Pad_D1.0mm, F.Cu at (42.5, 97.7)
- added TP25: TestPoint, TestPoint:TestPoint_Pad_D1.0mm, F.Cu at (60.9, 97.5)
- added TP27: TestPoint, TestPoint:TestPoint_Pad_D1.0mm, F.Cu at (46.0, 100.2)
- added TP28: TestPoint, TestPoint:TestPoint_Pad_D1.0mm, F.Cu at (58.6, 97.8)
- added TP29: TestPoint, TestPoint:TestPoint_Pad_D1.0mm, F.Cu at (37.4, 100.5)
- added TP30: TestPoint, TestPoint:TestPoint_Pad_D1.0mm, F.Cu at (60.8, 100.0)
- added TP32: TestPoint, TestPoint:TestPoint_Pad_D1.0mm, F.Cu at (35.1, 87.2)
- moved R5 0.55 mm to (43.7, 73.7)
- moved R64 0.55 mm to (43.7, 73.0)
- moved R8 0.55 mm to (43.7, 74.5)
- moved C5 0.20 mm to (38.7, 91.5)
- renumbered D19 to JTAG1, D16 to JTAG2, D17 to RX1, D14 to RX2, D18 to TX1, D15 to TX2
Routing:
- net /TMS_2: track 0.00 -> 44.8 mm, vias 0 -> 3
- net /TCK_1: track 0.00 -> 34.0 mm, vias 0 -> 2
- net /TDI_1: track 19.1 -> 50.8 mm, vias 1 -> 3
- net /TX_LED2: track 0.00 -> 24.5 mm, vias 0 -> 2
- net /RX_LED2: track 0.00 -> 24.1 mm, vias 0 -> 2
- net /JTAG_LED2: track 0.00 -> 22.7 mm, vias 0 -> 2
- net /JTAG_LED1: track 0.00 -> 20.7 mm, vias 0 -> 2
- net /TMS_1: track 11.2 -> 31.0 mm, vias 1 -> 3
- net /TXD_2: track 20.1 -> 37.8 mm, vias 1 -> 3
- net /NTRST_1: track 0.00 -> 11.4 mm, vias 0 -> 2
- net /VTREF_2: track 45.7 -> 55.7 mm
- net /RXD_2: track 9.94 -> 19.5 mm
- net /TDO_1: track 19.1 -> 28.1 mm, vias 1 -> 3
- net Net-(J1-D+-PadA6): track 2.30 -> 11.0 mm, vias 0 -> 2
- net Net-(J1-D--PadA7): track 2.30 -> 10.3 mm, vias 0 -> 2
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- added copper zone on In2.Cu, net /JTAG_LED1
- added copper zone on B.Cu, net /JTAG_LED2
- added copper zone on In2.Cu, net /NTRST_1
- added copper zone on In2.Cu, net /RX_LED2
- added copper zone on B.Cu, net /TCK_1
- added copper zone on B.Cu, net /TMS_2
- added copper zone on In2.Cu, net /TMS_2
- added copper zone on In2.Cu, net /TX_LED2
- added copper zone on In2.Cu, net Net-(J1-D+-PadA6)
- added copper zone on In2.Cu, net Net-(J1-D--PadA7)
Other:
- board text added: "FTDI_3V3_1"
- board text added: "FTDI_3V3_2"
- board text added: "GND"
- board text added: "RXD1"
- board text added: "RXD2"
- board text added: "TCK1"
- board text added: "TCK2"
- board text added: "TDI1"
- board text added: "TDI2"
- board text added: "TDO1"
- board text added: "TDO2"
- board text added: "TMS1"
- board text added: "TMS2"
- board text added: "TXD1"
- board text added: "TXD2"
- board text added: "VTREF1"
- board text added: "VTREF2"

Commit message: add: usb labels
Other:
- board text added: "Bitstream"
- board text added: "ELF"
Changed lines of the file:
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@@
 		(tags "USB C Type-C Receptacle SMD USB 2.0 16P 16C USB4105-15-A USB4105-15-A-060 USB4105-15-A-120 USB4105-GF-A USB4105-GF-A-060 USB4105-GF-A-120")
 		(property "Reference" "J2"
-			(at 6.3 0.11 270)
+			(at -5.9 2.41 270)
 			(unlocked yes)
 			(layer "F.SilkS")
@@
 		(tags "USB C Type-C Receptacle SMD USB 2.0 16P 16C USB4105-15-A USB4105-15-A-060 USB4105-15-A-120 USB4105-GF-A USB4105-GF-A-060 USB4105-GF-A-120")
 		(property "Reference" "J1"
-			(at -6.2 0.01 270)
+			(at 5.9 2.71 270)
 			(unlocked yes)
 			(layer "F.SilkS")
@@
 		(layer "Edge.Cuts")
 	)
+	(gr_text "ELF"
+		(at 28.7 67.3 0)
+		(layer "F.SilkS")
+		(effects
+			(font
+				(size 1 1)
+				(thickness 0.15)
+			)
+			(justify left bottom)
+		)
+	)
+	(gr_text "Bitstream"
+		(at 28.7 101.1 0)
+		(layer "F.SilkS")
+		(effects
+			(font
+				(size 1 1)
+				(thickness 0.15)
+			)
+			(justify left bottom)
+		)
+	)
 	(gr_text "GND"
