File: riskybirdv3_connector/riskybirdv3_connector.kicad_pcb (KiCad board)
At the start: 4 copper layers, 34.7 x 37 mm, 92 parts, among them J1 USB_C_Receptacle_USB2.0_16P, J2 USB_C_Receptacle_USB2.0_16P, J3 Conn_02x10_Odd_Even, U1 AP2112K-3.3, U15 FT2232HL-REEL, U2 AP2112K-3.3, U9 FT2232HL-REEL, Y2 f, Y3 f

Commit message: riskybirdv3 connector (programmer): VPLL/VPHY ferrites + 93LC66C EEPROM + design-rule sync
Programmer/connector board respin updates.

Schematic (riskybirdv3_connector.kicad_sch):
- Added VPLL/VPHY supply ferrites FB2-FB5 for FTDI PLL/PHY rail filtering.
- Removed the 22 ohm USB series resistors (direct USB D+/D- routing).
- Wired 93LC66C EEPROM (U3) for FTDI USB descriptor/config storage.
- LCSC part sync.

PCB (riskybirdv3_connector.kicad_pcb):
- Layout updated to match the ferrite/EEPROM/USB schematic changes.

Design rules:
- riskybirdv3_connector.kicad_dru + JLCPCB.kicad_dru synced from the
  base board's rule set.
Parts:
- removed R5, R6, R8, R9: 22R, Resistor_SMD:R_0201_0603Metric
- added C89: 100nF, Capacitor_SMD:C_0201_0603Metric, F.Cu at (43.6, 93.0)
- added C90: 4.7u, Capacitor_SMD:C_0402_1005Metric, F.Cu at (43.6, 93.9)
- added C91: 100nF, Capacitor_SMD:C_0201_0603Metric, F.Cu at (44.2, 75.0)
- added C92: 4.7u, Capacitor_SMD:C_0402_1005Metric, F.Cu at (42.9, 74.5)
- added C93: 100nF, Capacitor_SMD:C_0201_0603Metric, F.Cu at (45.0, 67.2)
- added C94: 4.7u, Capacitor_SMD:C_0402_1005Metric, F.Cu at (45.9, 67.0)
- added C95: 100nF, Capacitor_SMD:C_0201_0603Metric, F.Cu at (40.1, 89.9)
- added C96: 4.7u, Capacitor_SMD:C_0402_1005Metric, F.Cu at (39.3, 89.9)
- added C97: 100nF, Capacitor_SMD:C_0201_0603Metric, F.Cu at (56.3, 85.0)
- added FB2: 600R@100 MHz, Inductor_SMD:L_0603_1608Metric, B.Cu at (48.0, 94.1)
- added FB3: 600R@100 MHz, Inductor_SMD:L_0603_1608Metric, B.Cu at (48.2, 73.3)
- added FB4: 600R@100 MHz, Inductor_SMD:L_0603_1608Metric, B.Cu at (49.0, 71.1)
- added FB5: 600R@100 MHz, Inductor_SMD:L_0603_1608Metric, B.Cu at (49.5, 94.9)
- added JTAG3: LED_Red, LED_SMD:LED_0402_1005Metric, F.Cu at (32.6, 67.0)
- added JTAG4: LED_Red, LED_SMD:LED_0402_1005Metric, F.Cu at (30.7, 88.0)
- added R68: 150, Resistor_SMD:R_0201_0603Metric, F.Cu at (30.6, 87.1)
- added U3: 93LC66C, Package_SO:MSOP-8_3x3mm_P0.65mm, F.Cu at (60.0, 87.8)
- C3, C5: value 10u -> 2.2u
- C4, C6, C68, C70: value 10u -> 4.7u
- JTAG1, JTAG2: value LED -> LED_Red
- R66: value 1k -> 2.2k
- R67: value 1k -> 150
- RX1, RX2: value LED -> LED_Yellow
- TX1, TX2: value LED -> LED_Green
- moved R67 29.8 mm to (32.6, 66.2), turned to 180 degrees
- moved R66 23.9 mm to (60.9, 91.3), turned to 180 degrees
- moved TP30 0.45 mm to (60.6, 100.4)
- turned R10 to -90 degrees
Connections:
- J1 pad A6: Net-(J1-D+-PadA6) -> /USB_DP_1
- J1 pad A7: Net-(J1-D--PadA7) -> /USB_DM_1
- J1 pad B6: Net-(J1-D+-PadA6) -> /USB_DP_1
- J1 pad B7: Net-(J1-D--PadA7) -> /USB_DM_1
- J2 pad A6: Net-(J2-D+-PadA6) -> /USB_DP_2
- J2 pad A7: Net-(J2-D--PadA7) -> /USB_DM_2
- J2 pad B6: Net-(J2-D+-PadA6) -> /USB_DP_2
- J2 pad B7: Net-(J2-D--PadA7) -> /USB_DM_2
- R66 pad 1: /FTDI_3v3_1 -> Net-(U3-DO)
- R66 pad 2: Net-(U9-VPLL) -> Net-(U15-EEDATA)
- R67 pad 1: /FTDI_3v3_2 -> /5V_1
- R67 pad 2: Net-(U15-VPLL) -> Net-(JTAG3-A)
- U15 pad 4: /FTDI_3v3_2 -> Net-(U15-VPHY)
- U15 pad 61: /FTDI_3v3_2 -> Net-(U15-EEDATA)
- U15 pad 62: /FTDI_3v3_2 -> /SCLK_2
- U15 pad 63: /FTDI_3v3_2 -> Net-(U15-EECS)
- U9 pad 4: /FTDI_3v3_1 -> Net-(U9-VPHY)
Routing:
- net /TDO_2: track 40.2 -> 147.9 mm
- net /5V_2: track 8.23 -> 29.9 mm
- net Net-(U15-EEDATA): track 0.00 -> 19.3 mm, vias 0 -> 2
- net Net-(U15-EECS): track 0.00 -> 18.0 mm, vias 0 -> 2
- net /SCLK_2: track 0.00 -> 17.5 mm, vias 0 -> 2
- net /TXD_2: track 37.8 -> 53.7 mm
- net /USB_DP_2: track 2.46 -> 17.4 mm, vias 0 -> 2
- net /FTDI_3v3_2: track 49.3 -> 63.8 mm, vias 2 -> 4
- net Net-(J2-D+-PadA6): track 14.1 -> 0.00 mm, vias 2 -> 0
- net /USB_DM_2: track 2.38 -> 16.2 mm, vias 0 -> 2
- net Net-(J2-D--PadA7): track 13.1 -> 0.00 mm, vias 2 -> 0
- net Net-(U15-VPHY): track 0.00 -> 12.7 mm, vias 0 -> 1
- net /USB_DP_1: track 1.84 -> 14.1 mm, vias 0 -> 2
- net GND: track 131.8 -> 143.8 mm, vias 22 -> 25
- net /USB_DM_1: track 1.71 -> 13.1 mm, vias 0 -> 2
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- added copper zone on In2.Cu, net /USB_DM_1
- added copper zone on B.Cu, net /USB_DM_2
- added copper zone on In2.Cu, net /USB_DP_1
- added copper zone on B.Cu, net /USB_DP_2
- removed copper zone on In2.Cu, net /FTDI_3v3_2
- removed copper zone on In2.Cu, net Net-(J1-D+-PadA6)
- removed copper zone on In2.Cu, net Net-(J1-D--PadA7)
- removed copper zone on B.Cu, net Net-(J2-D+-PadA6)
- removed copper zone on B.Cu, net Net-(J2-D--PadA7)
Other:
- board text added: "Programmer V1.1"
