File: riskybirdv3_base/riskybirdv3.kicad_pcb (KiCad board)
At the start: 4 copper layers, 69.8 x 65 mm, 183 parts, among them IC1 PMW3901MB-TXQT, J1 USB_B_Micro, J10 Conn_01x05, J11 Conn_01x05, J13 Conn_02x12_Odd_Even_MountingP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, J18 Conn_01x05_MountingPin, J19 Conn_01x30_MountingPin, J2 Conn_01x05, J3 Conn_01x02, J4 Conn_01x02, J5 Conn_01x02, J6 Conn_01x02, J7 Conn_01x02, J8 USB_B_Micro, J9 Conn_01x05, Q1 SI2302, Q2 SI2302, Q3 SI2302, Q4 SI2302, Q8 BC847BDW1, SW1 SW_SPST, SW2 SW_SPST, SW3 SW_SPST, SW4 SW_SPST, U1 ADS7128IRTER, U10 TLV70018DCKR, U11 TPS54331D, U12 LP2985-3.0, U13 TPS2113A, U14 ESP32-C6-MINI-1/U, U3 BMI088, U4 MCP73831-2-OT, U6 FT2232HL-REEL, U7 TPS2113A, U8 FT231XS, U9 VL53L1CXV0FY1, Y1 f

Commit message: riskybirdv3: PMW3901 fixes (motor3 R, LED_N NC unroute, CamRST pull-up) + board
- Add missing MOTOR3 FPGA-leg series resistor (was ESP-only).
- Unroute PMW3901 pin 20 (datasheet NC; symbol mislabels it LED_N).
- CamRST/NRESET: add 47k pull-up to +3V3 (defaults sensor to running).
- Board (.kicad_pcb) current state.

TODO (power, next): SoM VIN wired to +5V (USB-only) -> must be +3V3;
B66_VCCO (bank 66 HP, JB3) not supplied; buck-boost size for >=4A SoM;
verify /VBAT -> JB1.80.
Parts:
- added C44: 0.1u, Capacitor_SMD:C_0402_1005Metric, F.Cu at (229.2, 111.8)
- added C45: 0.1u, Capacitor_SMD:C_0402_1005Metric, F.Cu at (229.2, 113.7)
- added C47: 10u, Capacitor_SMD:C_0402_1005Metric, F.Cu at (229.2, 115.7)
- added C48: 10u, Capacitor_SMD:C_0402_1005Metric, F.Cu at (229.2, 117.7)
- added C49: 10u, Capacitor_SMD:C_0402_1005Metric, F.Cu at (232.1, 111.8)
- added C50: 0.1u, Capacitor_SMD:C_0402_1005Metric, F.Cu at (232.1, 113.7)
- added C51: 0.1u, Capacitor_SMD:C_0402_1005Metric, F.Cu at (232.1, 115.7)
- added C52: 1u, Capacitor_SMD:C_0402_1005Metric, F.Cu at (232.1, 117.7)
- added C53: 1u, Capacitor_SMD:C_0402_1005Metric, F.Cu at (235.0, 111.8)
- added C54: 0.1u, Capacitor_SMD:C_0402_1005Metric, F.Cu at (235.0, 113.7)
- added C55: 1u, Capacitor_SMD:C_0402_1005Metric, F.Cu at (235.0, 115.7)
- added C57: 0.1u, Capacitor_SMD:C_0402_1005Metric, F.Cu at (235.0, 117.7)
- added C59: 1uF, Capacitor_SMD:C_0201_0603Metric, F.Cu at (219.2, 103.8)
- added C60: 0.1u, Capacitor_SMD:C_0201_0603Metric, F.Cu at (219.2, 105.5)
- added C61: 0.1u, Capacitor_SMD:C_0201_0603Metric, F.Cu at (219.2, 107.3)
- added C62: 0.1u, Capacitor_SMD:C_01005_0402Metric, F.Cu at (241.2, 111.6)
- added C63: 0.1u, Capacitor_SMD:C_1206_3216Metric, F.Cu at (250.8, 97.3)
- added C65: 4.7u, Capacitor_SMD:C_0201_0603Metric, F.Cu at (219.2, 109.0)
- added C66: 1uF, Capacitor_SMD:C_0201_0603Metric, F.Cu at (219.2, 110.8)
- added J1: Conn_02x10_Odd_Even, riskybird_lcsc:CONN-SMD_FTSH-110-01-L-DV-K-TR, F.Cu at (235.6, 106.9)
- added JB1: Conn_02x50_Odd_Even_Shielded, Connector_Samtec:Samtec_LSHM-150-xx.x-x-DV-S_2x50-1SH_P0.50mm_Vertical, F.Cu at (157.2, 107.4)
- added JB2: Conn_02x50_Odd_Even_Shielded, Connector_Samtec:Samtec_LSHM-150-xx.x-x-DV-S_2x50-1SH_P0.50mm_Vertical, F.Cu at (189.7, 107.7)
- added JB3: Conn_02x30_Odd_Even_Shielded, Connector_Samtec:Samtec_LSHM-130-xx.x-x-DV-S_2x30-1SH_P0.50mm_Vertical, F.Cu at (173.4, 87.8)
- added L4: 2.2u, Inductor_SMD:L_0603_1608Metric, F.Cu at (249.0, 117.2)
- added Q5: AON7407, riskybird_lcsc:DFN-8_L3.0-W3.0-P0.65-BL, F.Cu at (244.9, 115.1)
- added R10: 10k, Resistor_SMD:R_0201_0603Metric, F.Cu at (221.7, 105.5)
- added R13: 47R, Resistor_SMD:R_0201_0603Metric, F.Cu at (221.7, 107.3)
- added R14: 47R, Resistor_SMD:R_0201_0603Metric, F.Cu at (221.7, 109.0)
- added R17: 47R, Resistor_SMD:R_0201_0603Metric, F.Cu at (221.7, 110.8)
- added R18: 47R, Resistor_SMD:R_0201_0603Metric, F.Cu at (221.7, 112.5)
- added R21: 47R, Resistor_SMD:R_0201_0603Metric, F.Cu at (221.7, 114.3)
- added R24: 47R, Resistor_SMD:R_0201_0603Metric, F.Cu at (221.7, 116.0)
- added R26: 47R, Resistor_SMD:R_0201_0603Metric, F.Cu at (221.7, 117.8)
- added R27: 47R, Resistor_SMD:R_0201_0603Metric, F.Cu at (224.1, 103.8)
- added R28: 47R, Resistor_SMD:R_0201_0603Metric, F.Cu at (224.1, 105.5)
- added R29: 47R, Resistor_SMD:R_0201_0603Metric, F.Cu at (224.1, 107.3)
- added R34: 47R, Resistor_SMD:R_0201_0603Metric, F.Cu at (224.1, 109.0)
- added R35: 340k, Resistor_SMD:R_0201_0603Metric, F.Cu at (224.1, 110.8)
- added R36: 100k, Resistor_SMD:R_0201_0603Metric, F.Cu at (224.1, 112.5)
- added R37: 47k, Resistor_SMD:R_0201_0603Metric, F.Cu at (224.1, 114.3)
- added R38: 47R, Resistor_SMD:R_0201_0603Metric, F.Cu at (224.1, 116.0)
- added R4: 10k, Resistor_SMD:R_0201_0603Metric, F.Cu at (219.2, 112.5)
- added R45: 100k, Resistor_SMD:R_0201_0603Metric, F.Cu at (224.1, 117.8)
- added R58: 100k, Resistor_SMD:R_0201_0603Metric, F.Cu at (226.6, 103.8)
- added R59: 316k, Resistor_SMD:R_0201_0603Metric, F.Cu at (226.6, 105.5)
- added R6: 10k, Resistor_SMD:R_0201_0603Metric, F.Cu at (219.2, 114.3)
- added R60: 100k, Resistor_SMD:R_0201_0603Metric, F.Cu at (226.6, 107.3)
- added R61: 52.3k, Resistor_SMD:R_0201_0603Metric, F.Cu at (226.6, 109.0)
- added R62: 48.7k, Resistor_SMD:R_0201_0603Metric, F.Cu at (226.6, 110.8)
- added R63: 100, Resistor_SMD:R_0201_0603Metric, F.Cu at (226.6, 112.5)
- added R64: 100, Resistor_SMD:R_0201_0603Metric, F.Cu at (226.6, 114.3)
- added R65: 100, Resistor_SMD:R_0201_0603Metric, F.Cu at (226.6, 116.0)
- added R66: 100, Resistor_SMD:R_0201_0603Metric, F.Cu at (226.6, 117.8)
- added R7: 10k, Resistor_SMD:R_0201_0603Metric, F.Cu at (219.2, 116.0)
- added R8: 10k, Resistor_SMD:R_0201_0603Metric, F.Cu at (219.2, 117.8)
- added R9: 10k, Resistor_SMD:R_0201_0603Metric, F.Cu at (221.7, 103.8)
- added SW5: SW_SPST, Button_Switch_SMD:SW_SPDT_CK_JS102011SAQN, F.Cu at (248.2, 107.9)
- added U11: TLV70015DCKT, riskybird_lcsc:SC-70-5_L2.0-W1.3-P0.65-LS2.1-BR, F.Cu at (249.0, 114.3)
- added U2: LTC3119EUFD#TRPBF, riskybird_lcsc:QFN-28_L5.0-W4.0-P0.50-TL-EP, F.Cu at (245.1, 99.0)
- added U7: TLV70028DCKR, riskybird_lcsc:SC-70-5_L2.1-W1.3-P0.65-LS2.1-BL, F.Cu at (250.0, 100.7)
- added U8: TPS2117DRLR_C22399676, riskybird_lcsc:SOT-583-8_L2.1-W1.2-P0.50-LS1.6-BL, F.Cu at (238.3, 112.3)
- C37, C43, C56, C58: footprint Capacitor_SMD:C_0402_1005Metric -> Capacitor_SMD:C_0201_0603Metric
- R40, R51, R52, R55, R56, R57: footprint Resistor_SMD:R_0402_1005Metric -> Resistor_SMD:R_0201_0603Metric
Connections:
- J13 pad 1: unconnected-(J13-Pin_1-Pad1) -> GND
- J13 pad 10: unconnected-(J13-Pin_10-Pad10) -> GND
- J13 pad 11: unconnected-(J13-Pin_11-Pad11) -> +1V8
- J13 pad 12: unconnected-(J13-Pin_12-Pad12) -> +1V5
- J13 pad 13: unconnected-(J13-Pin_13-Pad13) -> GND
- J13 pad 14: unconnected-(J13-Pin_14-Pad14) -> /MCLK
- J13 pad 15: unconnected-(J13-Pin_15-Pad15) -> GND
- J13 pad 16: unconnected-(J13-Pin_16-Pad16) -> /PCLK
- J13 pad 17: unconnected-(J13-Pin_17-Pad17) -> /D0
- J13 pad 18: unconnected-(J13-Pin_18-Pad18) -> /D1
- J13 pad 19: unconnected-(J13-Pin_19-Pad19) -> /D2
- J13 pad 2: unconnected-(J13-Pin_2-Pad2) -> +2V8
- J13 pad 20: unconnected-(J13-Pin_20-Pad20) -> /D3
- J13 pad 21: unconnected-(J13-Pin_21-Pad21) -> /D4
- J13 pad 22: unconnected-(J13-Pin_22-Pad22) -> /D5
- J13 pad 23: unconnected-(J13-Pin_23-Pad23) -> /D6
- J13 pad 24: unconnected-(J13-Pin_24-Pad24) -> /D7
- J13 pad 3: unconnected-(J13-Pin_3-Pad3) -> GND
- J13 pad 4: unconnected-(J13-Pin_4-Pad4) -> /TRIG
- J13 pad 5: unconnected-(J13-Pin_5-Pad5) -> /FVLD
- J13 pad 6: unconnected-(J13-Pin_6-Pad6) -> /LVLD
- J13 pad 7: unconnected-(J13-Pin_7-Pad7) -> /SCL
- J13 pad 8: unconnected-(J13-Pin_8-Pad8) -> /SDA
- J13 pad 9: unconnected-(J13-Pin_9-Pad9) -> /INT
- Q1 pad 1: Net-(Q1-G) -> /MOTOR1
- Q2 pad 1: Net-(Q2-G) -> /MOTOR2
- Q3 pad 1: Net-(Q3-G) -> /MOTOR3
- Q4 pad 1: Net-(Q4-G) -> /MOTOR4
- R15 pad 1: Net-(Q1-G) -> /MOTOR1
- R16 pad 1: Net-(Q3-G) -> /MOTOR3
- R19 pad 1: Net-(Q2-G) -> /MOTOR2
- R20 pad 1: Net-(Q4-G) -> /MOTOR4
- U14 pad 15: /SCLK -> Net-(U14-MTCK/GPIO6/ADC1_CH6)
- U14 pad 16: /MOSI -> Net-(U14-MTDO/GPIO7)
- U14 pad 17: /UART1_TX_3V3 -> /USB_DN
- U14 pad 18: /UART1_RX_3V3 -> /USB_DP
- U14 pad 24: /MISO -> Net-(U14-GPIO18)
- U14 pad 25: /NCS -> Net-(U14-GPIO19)
- U14 pad 26: /MOTOR2 -> Net-(U14-GPIO20)
- U14 pad 27: /MOTOR1 -> Net-(U14-GPIO21)
- U14 pad 28: /MOTOR4 -> Net-(U14-GPIO22)
- U14 pad 29: /MOTOR3 -> Net-(U14-GPIO23)
- U14 pad 5: /CamRST -> unconnected-(U14-GPIO2/ADC1_CH2-Pad5)
- U14 pad 6: /LED_N -> unconnected-(U14-GPIO3/ADC1_CH3-Pad6)

Commit message: riskybirdv3: USB-C+ESD, camera FPC/I2C level-shift, SoM B2B power/control, compact power switch
- ESP native USB-C (J8): USBLC6 ESD array on D+/D-, 5.1k CC pulldowns, HRO Type-C footprint
- U14 -> ESP32-C6-MINI-1U footprint (external U.FL antenna, no PCB-antenna keepout)
- HM01B0 camera (J13): DVP wiring + AVDD/IOVDD/DVDD rails; PCA9306 (U12) level-shifts 1.8V SCCB <-> shared 3.3V I2C
- SoM B2B (JB1/2/3): VIN/3.3VIN on +3V3, VCCIO banks, control pull-ups (EN1/JTAGSEL/NOSEQ/PGOOD/RESIN), JTAG data + VREF_JTAG(0R)
- SW3 -> MINI MSK12C02 slide switch (now only gates the P-FET, ~50uA)
- new footprints: ESP32-C6-MINI-1U, SW-SMD_MSK12CO2
Parts:
- removed C18, C19, C20, C21, C22, C24, C25, C27, C29, C31, C33: 100nF, Capacitor_SMD:C_0201_0603Metric
- removed C23: 10uF, Capacitor_SMD:C_0201_0603Metric
- removed C26: 4.7u, Capacitor_SMD:C_0201_0603Metric
- removed C28, C30: 4.7uF, Capacitor_SMD:C_0201_0603Metric
- removed C32: 3.3uF, Capacitor_SMD:C_0201_0603Metric
- removed C34: 1u, Capacitor_SMD:C_0201_0603Metric
- removed C35: 0.1u, Capacitor_SMD:C_0402_1005Metric
- removed C36: 4.7u, Capacitor_SMD:C_0402_1005Metric
- removed the C44 at (233.4, 66.0)
- removed the C45 at (233.4, 68.0)
- removed the C47 at (95.7, 114.2)
- removed the C48 at (94.5, 107.8)
- removed the C49 at (100.0, 111.1)
- removed the C50 at (100.4, 110.0)
- removed the C51 at (90.8, 112.5)
- removed the C52 at (103.1, 112.6)
- removed the C53 at (103.1, 111.0)
- removed the C54 at (90.8, 113.2)
- removed the C55 at (90.8, 111.8)
- removed the C57 at (236.3, 62.1)
- removed the C59 at (236.3, 66.0)
- removed D10, D11, D12: LED, LED_SMD:LED_0402_1005Metric
- removed D13: LED_BLUE, LED_SMD:LED_0805_2012Metric_Pad1.15x1.40mm_HandSolder
- removed D14: BAT54J, Diode_SMD:D_SOD-323F
- removed D8, D9: SK6812MINI, LED_SMD:LED_SK6812MINI_PLCC4_3.5x3.5mm_P1.75mm
- removed FB1, FB2: 600R@100MHz/0.5A, Inductor_SMD:L_0603_1608Metric
- removed the FID1 at (231.8, 99.7)
- removed the J1 at (226.8, 60.4)
- removed J18: Conn_01x05_MountingPin, Connector_JST:JST_ZH_B5B-ZR_1x05_P1.50mm_Vertical
- removed J19: Conn_01x30_MountingPin, Connector_FFC-FPC:Hirose_FH12-30S-0.5SH_1x30-1MP_P0.50mm_Horizontal
- removed L3: 6.8uH, Inductor_SMD:L_0603_1608Metric
- removed Q8: BC847BDW1, Package_TO_SOT_SMD:SOT-363_SC-70-6
- removed the R10 at (250.3, 33.9)
- removed the R13 at (116.0, 111.5)
- removed the R14 at (89.2, 86.8)
- removed the R17 at (90.0, 111.6)
- removed the R18 at (109.8, 87.0)
- removed the R21 at (206.3, 60.2)
- removed the R24 at (206.3, 62.1)
- removed the R26 at (92.3, 110.8)
- removed the R27 at (83.0, 88.6)
- removed the R28 at (83.8, 88.6)
- removed the R29 at (82.2, 88.6)
- removed the R34 at (94.5, 103.0)
- removed the R35 at (206.3, 64.1)
- removed the R36 at (206.3, 66.1)
- removed the R37 at (99.1, 106.5)
- removed the R38 at (98.8, 104.3)
- removed the R4 at (250.3, 25.1)
- removed the R45 at (90.8, 109.8)
- removed R47: 29.4k, Resistor_SMD:R_0201_0603Metric
- removed R48: 10.2k, Resistor_SMD:R_0201_0603Metric
- removed R49: 3.24k, Resistor_SMD:R_0201_0603Metric
- removed R50, R54: 150, Resistor_SMD:R_0402_1005Metric
- removed R53: 10k, Resistor_SMD:R_0402_1005Metric
- removed the R6 at (250.3, 26.9)
- removed the R7 at (250.3, 28.6)
- removed the R8 at (250.3, 30.4)
- removed the R9 at (250.3, 32.1)
- removed SW3: SW_SPST, Button_Switch_SMD:SW_SPDT_CK_JS102011SAQN
- removed the U11 at (95.7, 111.0)
- removed U13: TPS2113A, Package_SO:TSSOP-8_4.4x3mm_P0.65mm
- removed the U7 at (94.3, 105.2)
- removed the U8 at (217.6, 62.4)
- removed Y1: f, riskybird:OSC_CSTNE12M0G550000R0
- added C64: 470p, Capacitor_SMD:C_0201_0603Metric, F.Cu at (110.7, 109.1)
- added C67: 10u, Capacitor_SMD:C_0402_1005Metric, F.Cu at (96.7, 102.7)
- added C68: 1u, Capacitor_SMD:C_0201_0603Metric, F.Cu at (30.9, 67.2)
- added C69: 1u, Capacitor_SMD:C_0201_0603Metric, F.Cu at (30.9, 68.9)
- added C70: 1u, Capacitor_SMD:C_0201_0603Metric, F.Cu at (30.9, 70.7)
- added C71: 0.1u, Capacitor_SMD:C_0402_1005Metric, F.Cu at (33.5, 67.3)
- added C72: 0.1u, Capacitor_SMD:C_0402_1005Metric, F.Cu at (33.5, 69.3)
- added C73: 10u, Capacitor_SMD:C_0402_1005Metric, F.Cu at (33.5, 71.2)
- added C74: 10u, Capacitor_SMD:C_0402_1005Metric, F.Cu at (33.5, 73.2)
- added C75: 10u, Capacitor_SMD:C_0402_1005Metric, F.Cu at (33.5, 75.2)
- added FID1: DroneFrame, riskybird:riskybird_frame, F.Cu at (74.3, -59.4)
- added FID1: DroneFrame, riskybird:riskybird_frame, F.Cu at (100.3, 99.5)
- added J4: Conn_01x02, Connector_Molex:Molex_PicoBlade_53048-0210_1x02_P1.25mm_Horizontal, B.Cu at (66.9, 95.5)
- added J5: Conn_01x02, Connector_Molex:Molex_PicoBlade_53048-0210_1x02_P1.25mm_Horizontal, B.Cu at (68.3, 104.3)
- added J7: Conn_01x02, Connector_PinHeader_2.00mm:PinHeader_1x02_P2.00mm_Vertical, F.Cu at (115.8, 26.5)
- added R67: 200k, Resistor_SMD:R_0201_0603Metric, F.Cu at (30.9, 75.9)
- added R68: 2.2k, Resistor_SMD:R_0201_0603Metric, F.Cu at (30.9, 77.7)
- added R69: 2.2k, Resistor_SMD:R_0201_0603Metric, F.Cu at (30.9, 79.4)
- C44, C45, C50: footprint Capacitor_SMD:C_0402_1005Metric -> Capacitor_SMD:C_0201_0603Metric
- C62: value 0.1u -> 10u; footprint Capacitor_SMD:C_01005_0402Metric -> Capacitor_SMD:C_0402_1005Metric
- C63: value 0.1u -> 150u
- C65: footprint Capacitor_SMD:C_0201_0603Metric -> Capacitor_SMD:C_0402_1005Metric
- J1: moved to B.Cu
- J8: value USB_B_Micro -> USB_C_Receptacle_USB2.0_16P; footprint Connector_USB:USB_Micro-B_Molex_47346-0001 -> Connector_USB:USB_C_Receptacle_HRO_TYPE-C-31-M-12
- R11: value 10k -> 5.1k; footprint Resistor_SMD:R_0402_1005Metric -> Resistor_SMD:R_0201_0603Metric
- R39: value 10k -> 0R; footprint Resistor_SMD:R_0402_1005Metric -> Resistor_SMD:R_0201_0603Metric
- R46: value 332k -> 0R; moved to F.Cu
- R5: value 12k -> 5.1k
- SW5: footprint Button_Switch_SMD:SW_SPDT_CK_JS102011SAQN -> riskybird_lcsc:SW-SMD_MSK12CO2
- U12: value LP2985-3.0 -> PCA9306DC; footprint Package_TO_SOT_SMD:SOT-23-5 -> Package_SO:VSSOP-8_2.3x2mm_P0.5mm
- U14: footprint RF_Module:ESP32-C6-MINI-1 -> riskybird_lcsc:ESP32-C6-MINI-1U
- U6: value FT2232HL-REEL -> USBLC6-2P6; footprint Package_QFP:LQFP-64_10x10mm_P0.5mm -> Package_TO_SOT_SMD:SOT-666
- moved U12 202.6 mm to (37.8, 68.2)
- moved SW5 180.4 mm to (68.0, 100.0), turned to -90 degrees
- moved R39 175.5 mm to (30.9, 72.4)
- moved C1 161.4 mm to (62.1, -66.4)
- moved C11 161.4 mm to (76.4, -65.5)
- moved C12 161.4 mm to (78.2, -65.5)
- moved C13 161.4 mm to (79.8, -64.4)
- moved C15 161.4 mm to (81.4, -65.1)
- moved C16 161.4 mm to (65.1, -65.2)
- moved C17 161.4 mm to (66.0, -66.6)
- moved C2 161.4 mm to (83.6, -71.1)
- moved C3 161.4 mm to (81.5, -47.2)
- moved C40 161.4 mm to (64.9, -72.1)
- moved C42 161.4 mm to (82.3, -68.9)
- moved C6 161.4 mm to (72.0, -64.0)
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- renumbered J13 to HM01B0_Conn1
Connections:
- HM01B0_Conn1 pad 7: /SCL -> /CAM_SCL
- HM01B0_Conn1 pad 8: /SDA -> /CAM_SDA
- J1 pad 1: /FPGA_VTREF -> +3V3
- J1 pad 9: /RV_VTREF -> +3V3
- JB1 pad 2: +5V -> +3V3
- JB1 pad 34: /Some_Top_Reset -> /CHIP_EN
- JB1 pad 4: +5V -> +3V3
- JB1 pad 55: unconnected-(JB1-Pin_55-Pad55) -> /SDA
- JB1 pad 57: unconnected-(JB1-Pin_57-Pad57) -> /SCL
- JB1 pad 6: +5V -> +3V3
- JB2 pad 1: +5V -> +3V3
- JB2 pad 10: unconnected-(JB2-Pin_10-Pad10) -> +1V8
- JB2 pad 21: /SDA -> unconnected-(JB2-Pin_21-Pad21)
- JB2 pad 23: /SCL -> unconnected-(JB2-Pin_23-Pad23)
- JB2 pad 3: +5V -> +3V3
- JB2 pad 31: /FLVD -> /FVLD
- JB2 pad 5: +5V -> +3V3
- JB2 pad 7: +5V -> +3V3
- JB2 pad 8: unconnected-(JB2-Pin_8-Pad8) -> +1V8
- JB2 pad 92: /FTDI_3v3_2 -> Net-(JB2-Pin_72-Pad92)
- R11 pad 1: +5V -> Net-(J8-CC1)
- R39 pad 1: +3V3_USB -> +3V3
- R39 pad 2: Net-(U13-VSNS) -> Net-(JB2-Pin_72-Pad92)
- R46 pad 1: VCOM -> GND
- R46 pad 2: Net-(U11-EN) -> Net-(JB1-Pin_8)
- R5 pad 1: Net-(U6-REF) -> Net-(J8-CC2)
- U12 pad 1: +5V -> GND
- U12 pad 2: GND -> +1V8
- U12 pad 3: +5V -> /CAM_SCL
- U12 pad 4: Net-(U12-BP) -> /CAM_SDA
- U12 pad 5: +3V3_USB -> /SDA
- U6 pad 1: GND -> Net-(J8-D+-PadA6)
- U6 pad 2: /FTDI_OSCI -> GND
- U6 pad 3: /FTDI_OSCO -> Net-(J8-D--PadA7)
- U6 pad 4: Net-(U6-VPHY) -> /USB_DN
- U6 pad 5: GND -> +5V
- U6 pad 6: Net-(U6-REF) -> /USB_DP
Other:
- board size 69.8 x 65 mm -> 69.8 x 53 mm

Commit message: riskybirdv3: board placement/frame-rotation checkpoint + battery power-gating
- Board placement + H-frame rotation exploration (current placed state)
- Standby-drain gating: LED (D4) and battery-sense divider gated low-side via 2N7002 FETs (Q6/Q7) off VCOM -> zero drain when SW3 off
- Removed always-on ESP +BATT sense divider (R51/R52); battery sense moved to ADS7128 (U1)
- SW3 -> MINI MSK12C02 slide switch in place
Parts:
- removed the J4 at (60.9, -71.7)
- removed the J5 at (61.8, -46.1)
- removed the J7 at (115.8, 26.5)
- removed the J7 at (56.4, -48.9)
- removed R51: 200k, Resistor_SMD:R_0201_0603Metric
- removed R52: 100k, Resistor_SMD:R_0201_0603Metric
- added J7: Conn_01x02, Connector_PinHeader_2.00mm:PinHeader_1x02_P2.00mm_Vertical, F.Cu at (80.0, 112.0)
- added Q6: 2N7002, Package_TO_SOT_SMD:SOT-23, F.Cu at (91.7, 94.1)
- added Q7: 2N7002, Package_TO_SOT_SMD:SOT-23, B.Cu at (109.2, 118.4)
- added R47: 200k, Resistor_SMD:R_0201_0603Metric, F.Cu at (94.0, 94.1)
- added R48: 200k, Resistor_SMD:R_0201_0603Metric, B.Cu at (110.5, 119.7)
- C1, C46, C56, C59, C66, C68, C69, C70, C71, C72, C73, C74, Q3, Q4, R1, R10, R12, R16, R2, R20, R26, R27, R28, R29, R34, R37, R38, R46, R6, R67, R68, R69, R9, U11, U12, U4, U7: moved to B.Cu
- C14: footprint Capacitor_SMD:C_0201_0603Metric -> Capacitor_SMD:C_0402_1005Metric
- C16, C17, C4, C5, C6, C7, C8, R22, R23, R3, R30, R31, R32, R33, SW2, U1, U3, U5: moved to F.Cu
- C51, C52, C55, C57: footprint Capacitor_SMD:C_0402_1005Metric -> Capacitor_SMD:C_0201_0603Metric; moved to B.Cu
- C53, C54: footprint Capacitor_SMD:C_0402_1005Metric -> Capacitor_SMD:C_0201_0603Metric
- moved D1 199.8 mm to (107.9, 121.6)
- moved D4 199.8 mm to (108.9, 121.6)
- moved R1 198.9 mm to (107.9, 120.8), turned to -90 degrees
- moved U4 198.7 mm to (100.0, 126.4), turned to 180 degrees
- moved R12 198.5 mm to (108.9, 120.8), turned to -90 degrees
- moved R2 196.6 mm to (98.6, 124.2), turned to 180 degrees
- moved C1 194.4 mm to (100.7, 124.2), turned to 0 degrees
- moved R3 181.1 mm to (102.7, 127.6), turned to 180 degrees
- moved R19 179.4 mm to (93.6, 130.0), turned to 180 degrees
- moved Q2 178.7 mm to (92.9, 132.2), turned to 90 degrees
- moved D7 178.1 mm to (101.8, 125.6), turned to -90 degrees
- moved R15 177.8 mm to (106.3, 130.0)
- moved Q1 176.4 mm to (107.1, 132.3), turned to 90 degrees
- moved D3 174.7 mm to (95.0, 126.0), turned to 180 degrees
- moved C41 173.1 mm to (96.9, 123.5), turned to 90 degrees
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Connections:
- D4 pad 1: GND -> Net-(D4-K)
- J1 pad 1: +3V3 -> GND
- J1 pad 10: /RV_TDO -> +3V3
- J1 pad 11: /RV_TCK -> GND
- J1 pad 12: GND -> /RV_TCK
- J1 pad 13: /RV_TMS -> /RV_TDI
- J1 pad 14: /RV_TDI -> /RV_TMS
- J1 pad 15: /RV_TRST -> /RV_UART_TX
- J1 pad 16: /RV_UART_TX -> /RV_TRST
- J1 pad 17: /RV_UART_RX -> /TSI_UART_TX
- J1 pad 18: /TSI_UART_TX -> /RV_UART_RX
- J1 pad 19: /TSI_UART_RX -> GND
- J1 pad 2: GND -> +3V3
- J1 pad 20: GND -> /TSI_UART_RX
- J1 pad 3: /FPGA_TCK -> GND
- J1 pad 4: GND -> /FPGA_TCK
- J1 pad 5: /FPGA_TMS -> /FPGA_TDO
- J1 pad 6: /FPGA_TDO -> /FPGA_TMS
- J1 pad 7: /FPGA_TDI -> /FPGA_PROG_B
- J1 pad 8: /FPGA_PROG_B -> /FPGA_TDI
- J1 pad 9: +3V3 -> /RV_TDO
- JB1 pad 34: /CHIP_EN -> /RST
- R30 pad 1: +3V3 -> +BATT
- R31 pad 2: GND -> Net-(Q6-D)
- U14 pad 12: /VSENSE -> unconnected-(U14-GPIO0/ADC1_CH0/XTAL_32K_P-Pad12)
Other:
- board size 69.8 x 53 mm -> 53 x 69.8 mm
