File: riskybirdv3_base/riskybirdv3.kicad_pcb (KiCad board)
At the start: 4 copper layers, 70 x 70.6 mm, 201 parts, among them IC1 PMW3901MB-TXQT, J1 Conn_02x10_Odd_Even, J10 Conn_01x05, J11 Conn_01x05, J12 Conn_01x02, J2 Conn_01x05, J3 Conn_01x02, J4 Conn_01x02, J5 Conn_01x02, J6 Conn_01x02, J7 Conn_01x02, J8 USB_C_Receptacle_USB2.0_16P, J9 Conn_01x05, Q1 SI2302, Q10 AON7534, Q2 SI2302, Q3 SI2302, Q4 SI2302, Q6 2N7002, Q7 2N7002, Q8 AON7534, Q9 AON7534, SW1 SW_SPST, SW2 SW_SPST, SW4 SW_SPST, SW5 SW_SPST, U1 ADS7128IRTER, U10 TLV70018DCKR, U11 TLV70015DCKT, U12 PCA9306DC, U13 LM74700, U14 ESP32-C6-MINI-1/U, U15 TPS552882QRPMRQ1, U16 TPS259824ONRGER, U3 BMI088, U4 MCP73831-2-OT, U5 BMP388, U6 USBLC6-2P6, U7 TLV70028DCKR, U8 LM66100DCK, U9 VL53L1CXV0FY1

Commit message: riskybirdv3: L2 SMD attr fix; IC1 populate; exclude 1x5 ToF-slot headers; silk fixes
- L2 (XAL7030-152MEC power inductor): footprint component-type attr
  through_hole -> smd. Its pads are SMD but were mislabeled THT, so JLC
  categorized it as through-hole -> off the SMT line / not rendered in the
  assembly preview (and it fell into the hand-solder bucket).
- IC1 (PMW3901): cleared a stale PCB-footprint DNP so it populates
  (schematic was already dnp=no; F8 "don't overwrite footprints" had left
  the footprint attribute out of sync).
- J2/J9/J10/J11 (1x5 ToF breakout slots): in_bom=no + exclude_from_bom,
  LCSC cleared (value kept as slot documentation) -- user-soldered, not
  JLC-assembled.
- Plus silkscreen clearance fixes.
Parts:
- moved G1 0.38 mm to (89.6, 80.5)
Changed lines of the file:
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@@
 			)
 		)
-		(attr smd dnp)
+		(attr smd)
 		(duplicate_pad_numbers_are_jumpers no)
 		(fp_line
@@
 			(at 0 1.43 90)
 			(layer "B.SilkS")
+			(hide yes)
 			(effects
 				(font
@@
 			)
 		)
-		(property "LCSC Part" "C962136"
-			(at 0 0 0)
-			(unlocked yes)
+		(property "Datasheet" ""
+			(at 0 0 90)
 			(layer "B.Fab")
 			(hide yes)
 			(effects
 				(font
-					(size 1 1)
-					(thickness 0.15)
+					(size 1.27 1.27)
 				)
 				(justify mirror)
 			)
 		)
-		(property "Datasheet" ""
+		(property "Description" ""
 			(at 0 0 90)
 			(layer "B.Fab")
@@
 			)
 		)
-		(property "Description" ""
-			(at 0 0 90)
+		(property "LCSC Part" "C962136"
+			(at 0 0 0)
+			(unlocked yes)
 			(layer "B.Fab")
 			(hide yes)
 			(effects
 				(font
-					(size 1.27 1.27)
+					(size 1 1)
+					(thickness 0.15)
 				)
 				(justify mirror)
@@
 	(footprint "LOGO"
 		(layer "B.Cu")
-		(at 89.45 80.8)
+		(at 89.6 80.45)
 		(property "Reference" "G1"
 			(at 0 0 0)
@@
 			)
 		)
-		(property "LCSC Part" "C492404"
+		(property "LCSC Part" ""
 			(at 0 0 0)
 			(unlocked yes)
@@
 			)
 		)
-		(attr through_hole)
+		(attr through_hole exclude_from_bom)
 		(duplicate_pad_numbers_are_jumpers no)
 		(fp_line
@@
 			)
 		)
-		(property "LCSC Part" "C492404"
+		(property "LCSC Part" ""
 			(at 0 0 0)
 			(unlocked yes)
@@
 			)
 		)
-		(attr through_hole)
+		(attr through_hole exclude_from_bom)
 		(duplicate_pad_numbers_are_jumpers no)
 		(fp_line
@@
 			)
 		)
-		(property "LCSC Part" "C492404"
+		(property "LCSC Part" ""
 			(at 0 0 0)
 			(unlocked yes)
@@
 			)
 		)
-		(attr through_hole)
+		(attr through_hole exclude_from_bom)
 		(duplicate_pad_numbers_are_jumpers no)
 		(fp_line
@@
 			)
 		)
-		(attr through_hole)
+		(attr smd)
 		(duplicate_pad_numbers_are_jumpers no)
 		(fp_line
@@
 			)
 		)
-		(property "LCSC Part" "C492404"
+		(property "LCSC Part" ""
 			(at 0 0 0)
 			(unlocked yes)
@@
 			)
 		)
-		(attr through_hole)
+		(attr through_hole exclude_from_bom)
 		(duplicate_pad_numbers_are_jumpers no)
 		(fp_line
@@
 	)
 	(gr_text "-"
-		(at 108.7 118.6 -180)
+		(at 108.35 118.75 -180)
 		(layer "B.SilkS")
 		(effects
@@
 	)
 	(segment
-		(start 83.65 113.765)
-		(end 83.65 114.959925)
-		(width 0.4)
+		(start 120.4 113.55)
+		(end 117.65 116.3)
+		(width 0.3)
+		(layer "F.Cu")
+		(net "AGND")
+	)
+	(segment
+		(start 117.65 116.3)
+		(end 116.035 116.3)
+		(width 0.3)
+		(layer "F.Cu")
+		(net "AGND")
+	)
+	(via
+		(at 120.4 113.55)
+		(size 0.55)
+		(drill 0.25)
+		(layers "F.Cu" "B.Cu")
+		(net "AGND")
+	)
+	(via
+		(at 116.035 116.3)
+		(size 0.55)
+		(drill 0.25)
+		(layers "F.Cu" "B.Cu")
+		(net "AGND")
+	)
+	(segment
+		(start 115.752254 118.85)
+		(end 115.55 118.647746)
+		(width 0.3)
 		(layer "B.Cu")
-		(net "/VCAP_BAT")
+		(net "AGND")
 	)
 	(segment
-		(start 84.590075 115.9)
-		(end 85.65 115.9)
-		(width 0.4)
+		(start 118.1 118.813173)
+		(end 117.538173 119.375)
+		(width 0.3)
 		(layer "B.Cu")
-		(net "/VCAP_BAT")
+		(net "AGND")
 	)
 	(segment
-		(start 83.65 114.959925)
-		(end 84.590075 115.9)
-		(width 0.4)
+		(start 115.75 116.3)
+		(end 116.035 116.3)
+		(width 0.3)
 		(layer "B.Cu")
-		(net "/VCAP_BAT")
+		(net "AGND")
 	)
 	(segment
-		(start 85.65 115.9)
-		(end 86.45 115.1)
-		(width 0.4)
+		(start 120.05 113.42)
+		(end 120.27 113.42)
+		(width 0.3)
 		(layer "B.Cu")
-		(net "/VCAP_BAT")
+		(net "AGND")
 	)
 	(segment
-		(start 86.45 115.1)
-		(end 87.4625 115.1)
-		(width 0.4)
+		(start 115.55 118.647746)
+		(end 115.55 116.5)
+		(width 0.3)
 		(layer "B.Cu")
-		(net "/VCAP_BAT")
+		(net "AGND")
+	)
+	(segment
+		(start 117.538173 119.375)
+		(end 117.075 119.375)
+		(width 0.3)
+		(layer "B.Cu")
+		(net "AGND")
+	)
+	(segment
+		(start 120.27 113.42)
+		(end 120.4 113.55)
+		(width 0.3)
+		(layer "B.Cu")
+		(net "AGND")
+	)
+	(segment
+		(start 116.67 118.4)
+		(end 116.67 117.7)
+		(width 0.3)
+		(layer "B.Cu")
+		(net "AGND")
+	)
+	(segment
+		(start 116.419999 118.85)
+		(end 115.752254 118.85)
+		(width 0.3)
+		(layer "B.Cu")
+		(net "AGND")
+	)
+	(segment
+		(start 116.67 117.7)
+		(end 116.7 117.67)
+		(width 0.3)
+		(layer "B.Cu")
+		(net "AGND")
+	)
+	(segment
+		(start 116.67 118.97)
+		(end 116.67 118.4)
+		(width 0.3)
+		(layer "B.Cu")
+		(net "AGND")
+	)
+	(segment
+		(start 115.55 116.5)
+		(end 115.75 116.3)
+		(width 0.3)
+		(layer "B.Cu")
+		(net "AGND")
+	)
+	(segment
+		(start 118.1 118.37)
+		(end 118.1 118.813173)
+		(width 0.3)
+		(layer "B.Cu")
+		(net "AGND")
+	)
+	(segment
+		(start 117.075 119.375)
+		(end 116.67 118.97)
+		(width 0.3)
+		(layer "B.Cu")
+		(net "AGND")
+	)
+	(segment
+		(start 116.67 118.4)
+		(end 116.67 118.599999)
+		(width 0.3)
+		(layer "B.Cu")
+		(net "AGND")
+	)
+	(segment
+		(start 116.67 118.599999)
+		(end 116.419999 118.85)
+		(width 0.3)
+		(layer "B.Cu")
+		(net "AGND")
 	)
 	(segment
@@
 	)
 	(segment
+		(start 83.65 113.765)
+		(end 83.65 114.959925)
+		(width 0.4)
+		(layer "B.Cu")
+		(net "/VCAP_BAT")
+	)
+	(segment
+		(start 84.590075 115.9)
+		(end 85.65 115.9)
+		(width 0.4)
+		(layer "B.Cu")
+		(net "/VCAP_BAT")
+	)
+	(segment
+		(start 83.65 114.959925)
+		(end 84.590075 115.9)
+		(width 0.4)
+		(layer "B.Cu")
+		(net "/VCAP_BAT")
+	)
+	(segment
+		(start 85.65 115.9)
+		(end 86.45 115.1)
+		(width 0.4)
+		(layer "B.Cu")
+		(net "/VCAP_BAT")
+	)
+	(segment
+		(start 86.45 115.1)
+		(end 87.4625 115.1)
+		(width 0.4)
+		(layer "B.Cu")
+		(net "/VCAP_BAT")
+	)
+	(segment
 		(start 88.847761 112.95)
 		(end 88.95 112.95)
@@
 	)
 	(segment
-		(start 120.4 113.55)
-		(end 117.65 116.3)
-		(width 0.3)
-		(layer "F.Cu")
-		(net "AGND")
-	)
-	(segment
-		(start 117.65 116.3)
-		(end 116.035 116.3)
-		(width 0.3)
-		(layer "F.Cu")
-		(net "AGND")
-	)
-	(via
-		(at 120.4 113.55)
-		(size 0.55)
-		(drill 0.25)
-		(layers "F.Cu" "B.Cu")
-		(net "AGND")
-	)
-	(via
-		(at 116.035 116.3)
-		(size 0.55)
-		(drill 0.25)
-		(layers "F.Cu" "B.Cu")
-		(net "AGND")
-	)
-	(segment
-		(start 115.752254 118.85)
-		(end 115.55 118.647746)
-		(width 0.3)
-		(layer "B.Cu")
-		(net "AGND")
-	)
-	(segment
-		(start 118.1 118.813173)
-		(end 117.538173 119.375)
-		(width 0.3)
-		(layer "B.Cu")
-		(net "AGND")
-	)
-	(segment
-		(start 115.75 116.3)
-		(end 116.035 116.3)
-		(width 0.3)
-		(layer "B.Cu")
-		(net "AGND")
-	)
-	(segment
-		(start 120.05 113.42)
-		(end 120.27 113.42)
-		(width 0.3)
-		(layer "B.Cu")
-		(net "AGND")
-	)
-	(segment
-		(start 115.55 118.647746)
-		(end 115.55 116.5)
-		(width 0.3)
-		(layer "B.Cu")
-		(net "AGND")
-	)
-	(segment
-		(start 117.538173 119.375)
-		(end 117.075 119.375)
-		(width 0.3)
-		(layer "B.Cu")
-		(net "AGND")
-	)
-	(segment
-		(start 120.27 113.42)
-		(end 120.4 113.55)
-		(width 0.3)
-		(layer "B.Cu")
-		(net "AGND")
-	)
-	(segment
-		(start 116.67 118.4)
-		(end 116.67 117.7)
-		(width 0.3)
-		(layer "B.Cu")
-		(net "AGND")
-	)
-	(segment
-		(start 116.419999 118.85)
-		(end 115.752254 118.85)
-		(width 0.3)
-		(layer "B.Cu")
-		(net "AGND")
-	)
-	(segment
-		(start 116.67 117.7)
-		(end 116.7 117.67)
-		(width 0.3)
-		(layer "B.Cu")
-		(net "AGND")
-	)
-	(segment
-		(start 116.67 118.97)
-		(end 116.67 118.4)
-		(width 0.3)
-		(layer "B.Cu")
-		(net "AGND")
-	)
-	(segment
-		(start 115.55 116.5)
-		(end 115.75 116.3)
-		(width 0.3)
-		(layer "B.Cu")
-		(net "AGND")
-	)
-	(segment
-		(start 118.1 118.37)
-		(end 118.1 118.813173)
-		(width 0.3)
-		(layer "B.Cu")
-		(net "AGND")
-	)
-	(segment
-		(start 117.075 119.375)
-		(end 116.67 118.97)
-		(width 0.3)
-		(layer "B.Cu")
-		(net "AGND")
-	)
-	(segment
-		(start 116.67 118.4)
-		(end 116.67 118.599999)
-		(width 0.3)
-		(layer "B.Cu")
-		(net "AGND")
-	)
-	(segment
-		(start 116.67 118.599999)
-		(end 116.419999 118.85)
-		(width 0.3)
-		(layer "B.Cu")
-		(net "AGND")
-	)
-	(segment
