File: riskybirdv3_base/riskybirdv3.kicad_sch (KiCad schematic)
At the start: 194 parts, among them IC1 PMW3901MB-TXQT, J1 Conn_02x10_Odd_Even, J10 Conn_01x05, J11 Conn_01x05, J12 Conn_01x02, J2 Conn_01x05, J3 Conn_01x02, J4 Conn_01x02, J5 Conn_01x02, J6 Conn_01x02, J7 Conn_01x02, J8 USB_C_Receptacle_USB2.0_16P, J9 Conn_01x05, Q1 SI2302, Q10 AON7534, Q2 SI2302, Q3 SI2302, Q4 SI2302, Q6 2N7002, Q7 2N7002, Q8 AON7534, Q9 AON7534, SW1 SW_SPST, SW2 SW_SPST, SW4 SW_SPST, SW5 SW_SPST, U1 ADS7128IRTER, U10 TLV70018DCKR, U11 TLV70015DCKT, U12 PCA9306DC, U13 LM74700, U14 ESP32-C6-MINI-1/U, U15 TPS552882QRPMRQ1, U16 TPS259824ONRGER, U3 BMI088, U4 MCP73831-2-OT, U5 BMP388, U6 USBLC6-2P6, U7 TLV70028DCKR, U8 LM66100DCK, U9 VL53L1CXV0FY1

Commit message: riskybirdv3: annotate missing LCSC parts (sch) + PCB F8 net update / J1-J2 ECO
Schematic: assigned LCSC Part to the 47 in-BOM parts that had none
(caps, LEDs, BAT54, 1x05 headers, SI2302/2N7002 FETs, R25, and
U1/U3/U6/U8/U9/U10/U12/U13) — values per docs/RESPIN_BOM_JLC.md.
Electrically neutral: the 185 electrical ERC violations are unchanged.
J7/J12 left as in_bom=no solder-pad connectors (battery lead / PSU override).

Board: F8 net update from the completed single-rail power routing, plus
J1/J2 footprint ECO tweaks. Footprint LCSC bindings are NOT yet synced
from the schematic (F8 was run with "don't overwrite footprints"), so the
PCB footprints still lack LCSC on those 47 + R35 — to be applied in a
follow-up direct patch that preserves the J1/J2 footprint edits.
Parts:
- removed L1: SRP1265A-2R2M, riskybird_lcsc:IND-SMD_L13.5-W12.5, symbol riskybird_lcsc:SRP1265A-2R2M
- added D8: LED, LED_SMD:LED_0402_1005Metric, symbol Device:LED
- added L2: XAL7030-152MEC, riskybird_lcsc:IND-SMD_L7.5-W7.5_XAL7030-152MEC, symbol riskybird_lcsc:XAL7030-152MEC
- added R35: 150, Resistor_SMD:R_0201_0603Metric, symbol Device:R
- added R58: 10k, Resistor_SMD:R_0201_0603Metric, symbol Device:R
- C11, C12, C86, C87: LCSC Part (none) -> C59461
- C14, C46, C47, C48, C49, C73, C74, C75, C85: LCSC Part (none) -> C15525
- C2, C3, C40, C41: LCSC Part (none) -> C140782
- C71, C72: LCSC Part (none) -> C1525
- C80: LCSC Part (none) -> C528968
- C81: value 100p -> 82p
- C82: value 8.2n -> 5.6n
- D1, D4: LCSC Part (none) -> C965793
- D2, D3, D5, D6: LCSC Part (none) -> C86299
- D7: LCSC Part (none) -> C25503345
- J10, J11, J2, J9: LCSC Part (none) -> C492404
- Q1, Q2, Q3, Q4: LCSC Part (none) -> C2891732
- Q6, Q7: LCSC Part (none) -> C8545
- R25: LCSC Part (none) -> C22356394
- R76: value 28.7k -> 19.6k
- R79: value 2.6k -> 3.65k
- U1: LCSC Part (none) -> C2867992
- U10: LCSC Part (none) -> C133796
- U12: LCSC Part (none) -> C33196
- U13: LCSC Part (none) -> C2941042
- U3: LCSC Part (none) -> C194919
- U6: LCSC Part (none) -> C2827693
- U8: LCSC Part (none) -> C5219211
- U9: LCSC Part (none) -> C190004
Connections:
- net +3V3: now also R35.1, R58.1
- net GPIO7: now also D8.1 (K)
- net GPIO9: now also R58.2
- net MOSI: now also R29.2; no longer R34.2
- net MOTION: now also JB1.65 (Pin_65); no longer JB2.73 (Pin_73)
- net SCLK: now also R34.2; no longer R29.2
- net TSI_UART_RX: now also JB1.18 (Pin_18); no longer JB3.60 (Pin_60)
- net TSI_UART_TX: now also JB1.20 (Pin_20); no longer JB3.59 (Pin_59)
- net at C78.2, Q10.5 (D), Q10.6 (D)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: now also L2.1
- net at C76.2, U15.21 (SW2), U15.25 (SW2): now also L2.2
- net at JB1.75 (Pin_75): now also R27.1
- net at JB1.77 (Pin_77): now also R28.1
- net at JB1.79 (Pin_79): now also R29.1
- net at JB1.81 (Pin_61): now also R34.1
- net at JB2.65 (Pin_65): no longer R29.1
- net at JB2.67 (Pin_67): no longer R34.1
- net at JB2.63 (Pin_63): no longer R28.1
- net at JB2.61 (Pin_61): no longer R27.1
- new net: D8.2 (A), R35.2
- no-connect marks 134 -> 127
Other:
- moved on the sheet: R55

Commit message: riskybirdv3: correct power-rail passive BOM + cap voltage uprate + AGND net-tie
Fixes a systemic copy-paste mis-annotation where 16 power-rail passives carried
the wrong LCSC/MPN (Value edited, part field left pointing at the source part).
Built as-is, JLC would have placed 100k for every set-point resistor and
1uF/100nF for the COMP + eFuse timing caps -> dead rail. Each now has the
correct part:
  R45/R78=40.2k C423536, R49=121 C474519, R50=604 C423470, R52=60.4k C473653,
  R74=57.6k C320974, R75/R77=27k C273283, R76=19.6k C423675, R79=3.65k C166220,
  R80=28k C473489, C81=82p C161439, C82=5.6n C3037635, C83=150p C384963,
  C84=22n C2880350.

Design edits from docs/RESPIN_POWER_VERIFY.md:
- R74 56.2k->57.6k: Vout 3.335->3.283V (whole band under TE0841 3.4V abs-max).
- VSYS/VSYS_FUSED Cin voltage uprate: C86/C87 22uF 6.3V->16V (C6119868),
  C49 10uF 0402 6.3V -> 10uF/16V 0603 (C962136, footprint resized+rerouted),
  C85 10uF 6.3V -> 4.7uF/25V 0402 (C2858031).
- C79 relabeled 4.7uF->1uF to match the accepted 1uF part (C53067).

Also: added the missing AGND<->GND net-tie footprint (NT1); synced all LCSC
bindings schematic->PCB footprints (48 added incl. R35, 15 updated),
J1/J2 footprints preserved.

Electrically neutral (185 ERC electrical violations unchanged); 0 value<->LCSC
mismatches; 0 in-BOM footprints missing LCSC.
Parts:
- added TP4: TestPoint, TestPoint:TestPoint_Pad_D1.0mm, symbol Connector:TestPoint
- C49: value 10u -> 10u/16V; footprint Capacitor_SMD:C_0402_1005Metric -> Capacitor_SMD:C_0603_1608Metric; LCSC Part C15525 -> C962136
- C79: value 4.7uF -> 1u
- C81: LCSC Part C53067 -> C161439; MPN CL03A105MQ3CSNH -> GRM0335C1H820JA01D
- C82: LCSC Part C53067 -> C3037635; MPN CL03A105MQ3CSNH -> 0201B562K500NT
- C83: LCSC Part C76928 -> C384963; MPN GRM033R60J104KE19D -> GRM0335C1H151FA01D
- C84: LCSC Part C76928 -> C2880350; MPN GRM033R60J104KE19D -> EMK063B7223KP-F
- C85: value 10u -> 4.7u/25V; LCSC Part C15525 -> C2858031
- C86, C87: value 22u -> 22u/16V; LCSC Part C59461 -> C6119868
- NT1: footprint (none) -> NetTie:NetTie-2_SMD_Pad0.5mm
- R45, R78: LCSC Part C270364 -> C423536; MPN 0201WMF1003TEE -> 0201WMF4022TEE
- R49: LCSC Part C270364 -> C474519; MPN 0201WMF1003TEE -> RC0201FR-07121RL
- R50: LCSC Part C270364 -> C423470; MPN 0201WMF1003TEE -> (none)
- R52: LCSC Part C270364 -> C473653; MPN 0201WMF1003TEE -> (none)
- R74: value 56.2k -> 57.6k; LCSC Part C270364 -> C320974; MPN 0201WMF1003TEE -> RC-01W5762FT
- R75, R77: LCSC Part C270364 -> C273283; MPN 0201WMF1003TEE -> RC0201FR-0727KL
- R76: LCSC Part C270364 -> C423675; MPN 0201WMF1003TEE -> 0201WMF1962TEE
- R79: LCSC Part C270364 -> C166220; MPN 0201WMF1003TEE -> RTT013651FTH
- R80: LCSC Part C270364 -> C473489; MPN 0201WMF1003TEE -> 0201WMF2802TEE
Connections:
- net GND: now also TP4.1

Commit message: riskybirdv3: L2 SMD attr fix; IC1 populate; exclude 1x5 ToF-slot headers; silk fixes
- L2 (XAL7030-152MEC power inductor): footprint component-type attr
  through_hole -> smd. Its pads are SMD but were mislabeled THT, so JLC
  categorized it as through-hole -> off the SMT line / not rendered in the
  assembly preview (and it fell into the hand-solder bucket).
- IC1 (PMW3901): cleared a stale PCB-footprint DNP so it populates
  (schematic was already dnp=no; F8 "don't overwrite footprints" had left
  the footprint attribute out of sync).
- J2/J9/J10/J11 (1x5 ToF breakout slots): in_bom=no + exclude_from_bom,
  LCSC cleared (value kept as slot documentation) -- user-soldered, not
  JLC-assembled.
- Plus silkscreen clearance fixes.
Parts:
- J10, J11, J2, J9: LCSC Part C492404 -> (none); now left out of the parts list
Changed lines of the file:
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@@
 		(body_style 1)
 		(exclude_from_sim no)
-		(in_bom yes)
+		(in_bom no)
 		(on_board yes)
 		(in_pos_files yes)
@@
 			)
 		)
-		(property "LCSC Part" "C492404"
+		(property "LCSC Part" ""
 			(at 0 0 0)
 			(hide yes)
@@
 		(body_style 1)
 		(exclude_from_sim no)
-		(in_bom yes)
+		(in_bom no)
 		(on_board yes)
 		(in_pos_files yes)
@@
 			)
 		)
-		(property "LCSC Part" "C492404"
+		(property "LCSC Part" ""
 			(at 0 0 0)
 			(hide yes)
@@
 		(body_style 1)
 		(exclude_from_sim no)
-		(in_bom yes)
+		(in_bom no)
 		(on_board yes)
 		(in_pos_files yes)
@@
 			)
 		)
-		(property "LCSC Part" "C492404"
+		(property "LCSC Part" ""
 			(at 0 0 0)
 			(hide yes)
@@
 		(body_style 1)
 		(exclude_from_sim no)
-		(in_bom yes)
+		(in_bom no)
 		(on_board yes)
 		(in_pos_files yes)
@@
 			)
 		)
-		(property "LCSC Part" "C492404"
+		(property "LCSC Part" ""
 			(at 0 0 0)
 			(hide yes)
